File: VREG_5V.kicad_pcb (KiCad board)
At the start: 2 copper layers, 25.4 x 25.4 mm, 7 parts, among them J1 USB_B, J2 Screw_Terminal_01x02, U1 LM7805_TO220

Commit message: 11.7.2025
Other:
- board text added: "7V~35V"
- board text added: "GND"
Changed lines of the file:
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@@
+		)
+	)
+	(gr_text "GND"
+		(at 164.084 76.581 180)
+		(layer "F.SilkS")
+		(effects
+			(font
+				(size 0.333333 1)
+				(thickness 0.083333)
+			)
+			(justify left bottom)
+		)
+	)
+	(gr_text "7V~35V"
+		(at 170.688 76.454 180)
+		(layer "F.SilkS")
+		(effects
+			(font
+				(size 0.333333 1)
+				(thickness 0.083333)
+			)
+			(justify left bottom)
 		)
 	)
